File: Design Files/Beacon32.sch (KiCad schematic (older format))
At the start: 40 parts, among them M1 ESP-WROOM-32, P1 CONN_01X01, P10 CONN_01X01, P11 CONN_01X01, P12 CONN_01X01, P13 CONN_01X01, P14 CONN_01X01, P15 CONN_01X01, P16 CONN_01X01, P17 CONN_01X02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

Commit message: Issue closed
Added Reset switch and RGB footprint changed
Parts:
- removed R1: 10K, Resistors_SMD:R_0603, symbol R-RESCUE-Alpine_swift
- removed U4: EE_Logo, EE:Logo_8, symbol EE_Logo
- added R1: 10k, Resistors_SMD:R_0603, symbol R
- added SW1: SW_PUSH, Explore:smd_push2_New, symbol SW_PUSH
- D3: symbol LED -> LED-RESCUE-Beacon32
- U3: footprint EE:Logo_8 -> Logo:Logo_8
- U7: footprint RGB LED:sfh5712 -> Explore:RGB_SMD_4pin_New
- Y1: footprint EE:SMD_RTC_Crstl -> Explore:SMD_RTC_Crstl
Connections:
- net +3V3: now also R1.1
- net EN: now also R1.2, SW1.2
- net GND: now also SW1.1
