File: Design Files/Beacon32.sch (KiCad schematic (older format))
At the start: 40 parts, among them M1 ESP-WROOM-32, P1 CONN_01X01, P10 CONN_01X01, P11 CONN_01X01, P12 CONN_01X01, P13 CONN_01X01, P14 CONN_01X01, P15 CONN_01X01, P16 CONN_01X01, P17 CONN_01X02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

Commit message: Drill Size Increased
Parts:
- P1, P10, P11, P12, P13, P14, P15, P16, P3, P4, P5, P6, P7, P8, P9: footprint Special pad:Specialpad -> pad:MinimaPad
Changed lines of the file:
@@
 F1 78 3C 1E CF 3E 80 1F 4C 3C 1E 8F C7 33 36 7E 30 F1 78 3C 1E CF D8 F8 C1 C4 E3 F1 78 3C 63 E3
 07 13 8F C7 E3 F1 8C 8D 1F 4C 3C 1E 8F C7 33 36 FB F2 60 62 CA 85 62 CB A6 E6 F1 78 3C 9E 06 FC
-17 A5 91 1A 44 2E AE 30 24 00 00 00 00 49 45 4E 44 AE 42 60 82 19
+17 A5 91 1A 44 2E AE 30 24 00 00 00 00 49 45 4E 44 AE 42 60 82
 EndData
 $EndBitmap
@@
 F 0 "P1" H 8290 1100 50  0000 C CNN
 F 1 "CONN_01X01" V 8270 1100 50  0001 C CNN
-F 2 "Special pad:Specialpad" H 8170 1100 50  0001 C CNN
+F 2 "pad:MinimaPad" H 8170 1100 50  0001 C CNN
 F 3 "" H 8170 1100 50  0000 C CNN
 	1    8170 1100
@@
 F 0 "P3" H 10280 1160 50  0000 C CNN
 F 1 "CONN_01X01" V 10270 1170 50  0001 C CNN
-F 2 "Special pad:Specialpad" H 10170 1170 50  0001 C CNN
+F 2 "pad:MinimaPad" H 10170 1170 50  0001 C CNN
 F 3 "" H 10170 1170 50  0000 C CNN
 	1    10170 1170
@@
 F 0 "P4" H 10030 900 50  0000 C CNN
 F 1 "CONN_01X01" V 10020 900 50  0001 C CNN
-F 2 "Special pad:Specialpad" H 9920 900 50  0001 C CNN
+F 2 "pad:MinimaPad" H 9920 900 50  0001 C CNN
 F 3 "" H 9920 900 50  0000 C CNN
 	1    9920 900
@@
 F 0 "P5" H 9660 2350 50  0000 C CNN
 F 1 "CONN_01X01" V 9660 2350 50  0001 C CNN
-F 2 "Special pad:Specialpad" H 9560 2350 50  0001 C CNN
+F 2 "pad:MinimaPad" H 9560 2350 50  0001 C CNN
 F 3 "" H 9560 2350 50  0000 C CNN
 	1    9560 2350
@@
 F 0 "P6" H 9350 690 50  0000 C CNN
 F 1 "CONN_01X01" V 9350 700 50  0001 C CNN
-F 2 "Special pad:Specialpad" H 9250 700 50  0001 C CNN
+F 2 "pad:MinimaPad" H 9250 700 50  0001 C CNN
 F 3 "" H 9250 700 50  0000 C CNN
 	1    9250 700
@@
 F 0 "P7" H 10040 1480 50  0000 C CNN
 F 1 "CONN_01X01" V 10040 1480 50  0001 C CNN
-F 2 "Special pad:Specialpad" H 9940 1480 50  0001 C CNN
+F 2 "pad:MinimaPad" H 9940 1480 50  0001 C CNN
 F 3 "" H 9940 1480 50  0000 C CNN
 	1    9940 1480
@@
 F 0 "P8" H 9830 1870 50  0000 C CNN
 F 1 "CONN_01X01" V 9830 1870 50  0001 C CNN
-F 2 "Special pad:Specialpad" H 9730 1870 50  0001 C CNN
+F 2 "pad:MinimaPad" H 9730 1870 50  0001 C CNN
 F 3 "" H 9730 1870 50  0000 C CNN
 	1    9730 1870
@@
 F 0 "P9" H 8070 1780 50  0000 C CNN
 F 1 "CONN_01X01" V 8070 1780 50  0001 C CNN
-F 2 "Special pad:Specialpad" H 7970 1780 50  0001 C CNN
+F 2 "pad:MinimaPad" H 7970 1780 50  0001 C CNN
 F 3 "" H 7970 1780 50  0000 C CNN
 	1    7970 1780
@@
 F 0 "P10" H 8170 1440 50  0000 C CNN
 F 1 "CONN_01X01" V 8150 1440 50  0001 C CNN
-F 2 "Special pad:Specialpad" H 8050 1440 50  0001 C CNN
+F 2 "pad:MinimaPad" H 8050 1440 50  0001 C CNN
 F 3 "" H 8050 1440 50  0000 C CNN
 	1    8050 1440
@@
 F 0 "P11" H 9750 2140 50  0000 C CNN
 F 1 "CONN_01X01" V 9730 2140 50  0001 C CNN
-F 2 "Special pad:Specialpad" H 9630 2140 50  0001 C CNN
+F 2 "pad:MinimaPad" H 9630 2140 50  0001 C CNN
 F 3 "" H 9630 2140 50  0000 C CNN
 	1    9630 2140
@@
 F 0 "P12" H 9370 2580 50  0000 C CNN
 F 1 "CONN_01X01" V 9350 2580 50  0001 C CNN
-F 2 "Special pad:Specialpad" H 9250 2580 50  0001 C CNN
+F 2 "pad:MinimaPad" H 9250 2580 50  0001 C CNN
 F 3 "" H 9250 2580 50  0000 C CNN
 	1    9250 2580
@@
 F 0 "P13" H 8580 2520 50  0000 C CNN
 F 1 "CONN_01X01" V 8560 2520 50  0001 C CNN
-F 2 "Special pad:Specialpad" H 8460 2520 50  0001 C CNN
+F 2 "pad:MinimaPad" H 8460 2520 50  0001 C CNN
 F 3 "" H 8460 2520 50  0000 C CNN
 	1    8460 2520
@@
 F 0 "P14" H 8430 2270 50  0000 C CNN
 F 1 "CONN_01X01" V 8410 2270 50  0001 C CNN
-F 2 "Special pad:Specialpad" H 8310 2270 50  0001 C CNN
+F 2 "pad:MinimaPad" H 8310 2270 50  0001 C CNN
 F 3 "" H 8310 2270 50  0000 C CNN
 	1    8310 2270
@@
 F 0 "P15" H 8270 2040 50  0000 C CNN
 F 1 "CONN_01X01" V 8250 2030 50  0001 C CNN
-F 2 "Special pad:Specialpad" H 8150 2030 50  0001 C CNN
+F 2 "pad:MinimaPad" H 8150 2030 50  0001 C CNN
 F 3 "" H 8150 2030 50  0000 C CNN
 	1    8150 2030
@@
 F 0 "P16" H 8830 840 50  0000 C CNN
 F 1 "CONN_01X01" V 8810 840 50  0001 C CNN
-F 2 "Special pad:Specialpad" H 8710 840 50  0001 C CNN
+F 2 "pad:MinimaPad" H 8710 840 50  0001 C CNN
 F 3 "" H 8710 840 50  0000 C CNN
 	1    8710 840

Commit message: Resized pads to 3.5mm
Parts:
- P1, P10, P11, P12, P13, P14, P15, P16, P3, P4, P5, P6, P7, P8, P9: footprint pad:MinimaPad -> pad:MinimaPad_3.5mm
Changed lines of the file:
@@
 F 0 "P1" H 8290 1100 50  0000 C CNN
 F 1 "CONN_01X01" V 8270 1100 50  0001 C CNN
-F 2 "pad:MinimaPad" H 8170 1100 50  0001 C CNN
+F 2 "pad:MinimaPad_3.5mm" H 8170 1100 50  0001 C CNN
 F 3 "" H 8170 1100 50  0000 C CNN
 	1    8170 1100
@@
 F 0 "P3" H 10280 1160 50  0000 C CNN
 F 1 "CONN_01X01" V 10270 1170 50  0001 C CNN
-F 2 "pad:MinimaPad" H 10170 1170 50  0001 C CNN
+F 2 "pad:MinimaPad_3.5mm" H 10170 1170 50  0001 C CNN
 F 3 "" H 10170 1170 50  0000 C CNN
 	1    10170 1170
@@
 F 0 "P4" H 10030 900 50  0000 C CNN
 F 1 "CONN_01X01" V 10020 900 50  0001 C CNN
-F 2 "pad:MinimaPad" H 9920 900 50  0001 C CNN
+F 2 "pad:MinimaPad_3.5mm" H 9920 900 50  0001 C CNN
 F 3 "" H 9920 900 50  0000 C CNN
 	1    9920 900
@@
 F 0 "P5" H 9660 2350 50  0000 C CNN
 F 1 "CONN_01X01" V 9660 2350 50  0001 C CNN
-F 2 "pad:MinimaPad" H 9560 2350 50  0001 C CNN
+F 2 "pad:MinimaPad_3.5mm" H 9560 2350 50  0001 C CNN
 F 3 "" H 9560 2350 50  0000 C CNN
 	1    9560 2350
@@
 F 0 "P6" H 9350 690 50  0000 C CNN
 F 1 "CONN_01X01" V 9350 700 50  0001 C CNN
-F 2 "pad:MinimaPad" H 9250 700 50  0001 C CNN
+F 2 "pad:MinimaPad_3.5mm" H 9250 700 50  0001 C CNN
 F 3 "" H 9250 700 50  0000 C CNN
 	1    9250 700
@@
 F 0 "P7" H 10040 1480 50  0000 C CNN
 F 1 "CONN_01X01" V 10040 1480 50  0001 C CNN
-F 2 "pad:MinimaPad" H 9940 1480 50  0001 C CNN
+F 2 "pad:MinimaPad_3.5mm" H 9940 1480 50  0001 C CNN
 F 3 "" H 9940 1480 50  0000 C CNN
 	1    9940 1480
@@
 F 0 "P8" H 9830 1870 50  0000 C CNN
 F 1 "CONN_01X01" V 9830 1870 50  0001 C CNN
-F 2 "pad:MinimaPad" H 9730 1870 50  0001 C CNN
+F 2 "pad:MinimaPad_3.5mm" H 9730 1870 50  0001 C CNN
 F 3 "" H 9730 1870 50  0000 C CNN
 	1    9730 1870
@@
 F 0 "P9" H 8070 1780 50  0000 C CNN
 F 1 "CONN_01X01" V 8070 1780 50  0001 C CNN
-F 2 "pad:MinimaPad" H 7970 1780 50  0001 C CNN
+F 2 "pad:MinimaPad_3.5mm" H 7970 1780 50  0001 C CNN
 F 3 "" H 7970 1780 50  0000 C CNN
 	1    7970 1780
@@
 F 0 "P10" H 8170 1440 50  0000 C CNN
 F 1 "CONN_01X01" V 8150 1440 50  0001 C CNN
-F 2 "pad:MinimaPad" H 8050 1440 50  0001 C CNN
+F 2 "pad:MinimaPad_3.5mm" H 8050 1440 50  0001 C CNN
 F 3 "" H 8050 1440 50  0000 C CNN
 	1    8050 1440
@@
 F 0 "P11" H 9750 2140 50  0000 C CNN
 F 1 "CONN_01X01" V 9730 2140 50  0001 C CNN
-F 2 "pad:MinimaPad" H 9630 2140 50  0001 C CNN
+F 2 "pad:MinimaPad_3.5mm" H 9630 2140 50  0001 C CNN
 F 3 "" H 9630 2140 50  0000 C CNN
 	1    9630 2140
@@
 F 0 "P12" H 9370 2580 50  0000 C CNN
 F 1 "CONN_01X01" V 9350 2580 50  0001 C CNN
-F 2 "pad:MinimaPad" H 9250 2580 50  0001 C CNN
+F 2 "pad:MinimaPad_3.5mm" H 9250 2580 50  0001 C CNN
 F 3 "" H 9250 2580 50  0000 C CNN
 	1    9250 2580
@@
 F 0 "P13" H 8580 2520 50  0000 C CNN
 F 1 "CONN_01X01" V 8560 2520 50  0001 C CNN
-F 2 "pad:MinimaPad" H 8460 2520 50  0001 C CNN
+F 2 "pad:MinimaPad_3.5mm" H 8460 2520 50  0001 C CNN
 F 3 "" H 8460 2520 50  0000 C CNN
 	1    8460 2520
@@
 F 0 "P14" H 8430 2270 50  0000 C CNN
 F 1 "CONN_01X01" V 8410 2270 50  0001 C CNN
-F 2 "pad:MinimaPad" H 8310 2270 50  0001 C CNN
+F 2 "pad:MinimaPad_3.5mm" H 8310 2270 50  0001 C CNN
 F 3 "" H 8310 2270 50  0000 C CNN
 	1    8310 2270
@@
 F 0 "P15" H 8270 2040 50  0000 C CNN
 F 1 "CONN_01X01" V 8250 2030 50  0001 C CNN
-F 2 "pad:MinimaPad" H 8150 2030 50  0001 C CNN
+F 2 "pad:MinimaPad_3.5mm" H 8150 2030 50  0001 C CNN
 F 3 "" H 8150 2030 50  0000 C CNN
 	1    8150 2030
@@
 F 0 "P16" H 8830 840 50  0000 C CNN
 F 1 "CONN_01X01" V 8810 840 50  0001 C CNN
-F 2 "pad:MinimaPad" H 8710 840 50  0001 C CNN
+F 2 "pad:MinimaPad_3.5mm" H 8710 840 50  0001 C CNN
 F 3 "" H 8710 840 50  0000 C CNN
 	1    8710 840
